Commit message: mesh generation finished

File: gazebo/launch/empty.xacro (robot description, xacro)
@@ -2,5 +2,5 @@
 <sdf version="1.4">
   <world name="default" xmlns:xacro="http://www.ros.org/wiki/xacro">
-    <xacro:property name="world_path" value="$(find utils_gdal)/res" />
+    <xacro:property name="utils_gdal_res" value="$(find utils_gdal)/res" />
     <!-- A global light source -->
     <include>
@@ -12,5 +12,6 @@
     </include>
     <plugin filename="libgazebo_dxf_map_plugin.so" name="gazebo_dxf">
-      <map>${world_path}/test.dxf</map>
+      <map>${utils_gdal_res}/walls.dxf</map>
+      <mesh_common>${utils_gdal_res}/mesh_common.dae</mesh_common>
     </plugin>
   </world>

Commit message: finished

File: gazebo/launch/empty.xacro (robot description, xacro)
@@ -14,4 +14,8 @@
       <map>${utils_gdal_res}/walls.dxf</map>
       <mesh_common>${utils_gdal_res}/mesh_common.dae</mesh_common>
+      <material>BlueTransparent</material>
+      <height>2.0</height>
+      <mesh_name>map</mesh_name>
+      <debug_sphere>false</debug_sphere>
     </plugin>
   </world>

Commit message: renderer got fix

File: gazebo/launch/empty.xacro (robot description, xacro)
@@ -2,5 +2,5 @@
 <sdf version="1.4">
   <world name="default" xmlns:xacro="http://www.ros.org/wiki/xacro">
-    <xacro:property name="utils_gdal_res" value="$(find utils_gdal)/res" />
+    <xacro:property name="cslibs_gdal_res" value="$(find cslibs_gdal)/res" />
     <!-- A global light source -->
     <include>
@@ -12,6 +12,6 @@
     </include>
     <plugin filename="libgazebo_dxf_map_plugin.so" name="gazebo_dxf">
-      <map>${utils_gdal_res}/walls.dxf</map>
-      <mesh_common>${utils_gdal_res}/mesh_common.dae</mesh_common>
+      <map>${cslibs_gdal_res}/walls.dxf</map>
+      <mesh_common>${cslibs_gdal_res}/mesh_common.dae</mesh_common>
       <material>BlueTransparent</material>
       <height>2.0</height>

Commit message: updating the gazebo dependencies

File: gazebo/launch/empty.xacro (robot description, xacro)
@@ -2,5 +2,5 @@
 <sdf version="1.4">
   <world name="default" xmlns:xacro="http://www.ros.org/wiki/xacro">
-    <xacro:property name="cslibs_gdal_res" value="$(find cslibs_gdal)/res" />
+    <xacro:property name="cslibs_vectormaps_res" value="$(find cslibs_vectormaps)/res" />
     <!-- A global light source -->
     <include>
@@ -12,6 +12,6 @@
     </include>
     <plugin filename="libcslibs_gdal_gazebo_dxf_map_plugin.so" name="gazebo_dxf">
-      <map>${cslibs_gdal_res}/walls.dxf</map>
-      <mesh_common>${cslibs_gdal_res}/mesh_common.dae</mesh_common>
+      <map>${cslibs_vectormaps_res}/walls.dxf</map>
+      <mesh_common>${cslibs_vectormaps_res}/mesh_common.dae</mesh_common>
       <material>BlueTransparent</material>
       <height>2.0</height>
